File: schematic/RC_Controller/rc_controller_basic/rc_controller_transmitter_comp.sch (EAGLE design)
At the start: 16 parts, among them IC1 ATMEGA328-20P, SW1 CT10-XXXX-A2

Commit message: updated schematics
Parts:
- added G1: AB9V, battery:AB9V
- added LED6, LED7: LEDLUMILED, led-lumiled:LEDLUMILED
- added SW2: CT10-XXXX-A2, switch-coto:CT10-XXXX-A2
- C3: value (none) -> 0.1uF
- Q1: value (none) -> 16MHz
- R1: value (none) -> 10k
Connections:
- removed net N$2: LED1.C, LED2.C, LED3.C, LED4.C, LED5.C, SW1.1
- new net N$11: G1.+, SW2.2
- new net N$14: IC1.(PCI22/AIN0OC0A)PD6, LED7.A
- new net N$15: LED1.C, LED2.C, LED3.C, LED4.C, LED5.C, LED6.C, LED7.C, SW1.1
- new net N$6: IC1.(PCI23/AIN1)PD7, LED6.A
- new net N$8: SW2.1, U$1.VCC
- net GND: now also G1.-
- net VCC: no longer U$1.VCC
Other:
- moved on the sheet: LED1, LED2, LED3, LED4, LED5, SW1
